File: UHF panel minus Y.kicad_sch (KiCad schematic)
At the start: 30 parts, among them IC1 LMT84DCKT, J1 CONSMA001-SMD-G, J2 2pin_header, J3 2pin_header, J4 2pin_header, T1 NCS1.5-232+, U1 AQZ10X, U2 S16008-33

Commit message: Fix solar cell connections
Other:
- note added: "Solar Cells"
- moved on the sheet: D1
Changed lines of the file:
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@@
 		)
 	)
+	(text "Solar Cells"
+		(exclude_from_sim no)
+		(at 22.352 102.362 90)
+		(effects
+			(font
+				(size 2.54 2.159)
+				(thickness 0.4318)
+				(bold yes)
+			)
+			(justify left bottom)
+		)
+	)
 	(text "Temperature sensor"
 		(exclude_from_sim no)
@@
 	)
 	(junction
-		(at 26.67 153.67)
+		(at 31.75 153.67)
 		(diameter 0)
 		(color 0 0 0 0)
@@
 	)
 	(junction
-		(at 26.67 162.56)
+		(at 31.75 162.56)
 		(diameter 0)
 		(color 0 0 0 0)
@@
 	)
 	(junction
-		(at 26.67 119.38)
+		(at 31.75 119.38)
 		(diameter 0)
 		(color 0 0 0 0)
@@
 	(wire
 		(pts
-			(xy 26.67 119.38) (xy 50.8 119.38)
+			(xy 31.75 119.38) (xy 55.88 119.38)
 		)
 		(stroke
@@
 	(wire
 		(pts
-			(xy 26.67 106.68) (xy 26.67 119.38)
+			(xy 31.75 106.68) (xy 31.75 119.38)
 		)
 		(stroke
@@
 	(wire
 		(pts
-			(xy 50.8 119.38) (xy 50.8 128.27)
+			(xy 55.88 119.38) (xy 55.88 128.27)
 		)
 		(stroke
@@
 	(wire
 		(pts
-			(xy 26.67 67.31) (xy 26.67 81.28)
+			(xy 31.75 67.31) (xy 31.75 81.28)
 		)
 		(stroke
@@
 	(wire
 		(pts
-			(xy 50.8 143.51) (xy 50.8 153.67)
+			(xy 55.88 143.51) (xy 55.88 153.67)
 		)
 		(stroke
@@
 	(wire
 		(pts
-			(xy 34.29 162.56) (xy 34.29 160.02)
+			(xy 39.37 162.56) (xy 39.37 160.02)
 		)
 		(stroke
@@
 	(wire
 		(pts
-			(xy 26.67 162.56) (xy 26.67 165.1)
+			(xy 31.75 162.56) (xy 31.75 165.1)
 		)
 		(stroke
@@
 	(wire
 		(pts
-			(xy 26.67 162.56) (xy 34.29 162.56)
+			(xy 31.75 162.56) (xy 39.37 162.56)
 		)
 		(stroke
@@
 	(wire
 		(pts
-			(xy 26.67 19.05) (xy 26.67 41.91)
+			(xy 31.75 19.05) (xy 31.75 41.91)
 		)
 		(stroke
@@
 	(wire
 		(pts
-			(xy 26.67 19.05) (xy 220.98 19.05)
+			(xy 31.75 19.05) (xy 220.98 19.05)
 		)
 		(stroke
@@
 	(wire
 		(pts
-			(xy 50.8 153.67) (xy 26.67 153.67)
+			(xy 55.88 153.67) (xy 31.75 153.67)
 		)
 		(stroke
@@
 	(wire
 		(pts
-			(xy 26.67 119.38) (xy 26.67 123.19)
+			(xy 31.75 119.38) (xy 31.75 123.19)
 		)
 		(stroke
@@
 	(wire
 		(pts
-			(xy 26.67 153.67) (xy 26.67 162.56)
+			(xy 31.75 153.67) (xy 31.75 162.56)
 		)
 		(stroke
@@
 	(wire
 		(pts
-			(xy 26.67 148.59) (xy 26.67 153.67)
+			(xy 31.75 148.59) (xy 31.75 153.67)
 		)
 		(stroke
@@
 	)
 	(label "VA"
-		(at 26.67 39.37 0)
+		(at 31.75 39.37 0)
 		(effects
 			(font
@@
 	)
 	(label "VC"
-		(at 26.67 113.03 0)
+		(at 31.75 113.03 0)
 		(effects
 			(font
@@
 	)
 	(label "VB"
-		(at 26.67 76.2 0)
+		(at 31.75 76.2 0)
 		(effects
 			(font
@@
 	(symbol
 		(lib_id "Custom-Symbols:Solar_cell_C")
-		(at 26.67 135.89 0)
+		(at 31.75 135.89 0)
 		(unit 1)
 		(exclude_from_sim no)
@@
 		(fields_autoplaced yes)
 		(property "Reference" "S1"
-			(at 21.59 135.89 0)
+			(at 26.67 135.89 0)
 			(effects
 				(font
@@
 		)
 		(property "Value" "Solar_cell_C"
-			(at 16.256 143.002 0)
+			(at 21.336 143.002 0)
 			(effects
 				(font
@@
 		)
 		(property "Footprint" "Custom-Footprints:solar_cell_C"
-			(at 14.478 129.794 0)
+			(at 19.558 129.794 0)
 			(effects
 				(font
@@
 		)
 		(property "Datasheet" ""
-			(at 26.67 135.89 0)
+			(at 31.75 135.89 0)
 			(effects
 				(font
@@
 		)
 		(property "Description" ""
-			(at 26.67 135.89 0)
+			(at 31.75 135.89 0)
 			(effects
 				(font
@@
 	(symbol
 		(lib_id "Custom-Symbols:solar_cell_B")
-		(at 26.67 93.98 0)
+		(at 31.75 93.98 0)
 		(unit 1)
 		(exclude_from_sim no)
@@
 		(fields_autoplaced yes)
 		(property "Reference" "S2"
-			(at 21.59 93.98 0)
+			(at 26.67 93.98 0)
 			(effects
 				(font
@@
 		)
 		(property "Value" "solar_cell_B"
-			(at 18.542 99.568 0)
+			(at 23.622 99.568 0)
 			(effects
 				(font
@@
 		)
 		(property "Footprint" "Custom-Footprints:solar_cell_B"
-			(at 16.002 87.376 0)
+			(at 21.082 87.376 0)
 			(effects
 				(font
@@
 		)
 		(property "Datasheet" ""
-			(at 26.67 93.98 0)
+			(at 31.75 93.98 0)
 			(effects
 				(font
@@
 		)
 		(property "Description" ""
-			(at 26.67 93.98 0)
+			(at 31.75 93.98 0)
 			(effects
 				(font
@@
 	(symbol
 		(lib_id "Custom-Symbols:CUHS20S30,H3F")
-		(at 50.8 137.16 0)
+		(at 55.88 137.16 0)
 		(unit 1)
 		(exclude_from_sim no)
@@
 		(fields_autoplaced yes)
 		(property "Reference" "D1"
-			(at 54.61 133.985 0)
+			(at 59.69 133.985 0)
 			(effects
 				(font
@@
 		)
 		(property "Value" "CUHS20S30,H3F"
-			(at 54.61 137.795 0)
+			(at 59.69 137.795 0)
 			(effects
 				(font
@@
 		)
 		(property "Footprint" "Custom-Footprints:CUHS20S30,H3F"
-			(at 26.416 137.922 0)
+			(at 31.496 137.922 0)
 			(effects
 				(font
@@
 		)
 		(property "Datasheet" ""
-			(at 50.8 137.16 0)
+			(at 55.88 137.16 0)
 			(effects
 				(font
@@
 		)
 		(property "Description" ""
-			(at 50.8 137.16 0)
+			(at 55.88 137.16 0)
 			(effects
 				(font
@@
 	(symbol
 		(lib_id "power:GND")
-		(at 26.67 165.1 0)
+		(at 31.75 165.1 0)
 		(unit 1)
 		(exclude_from_sim no)
@@
 		(fields_autoplaced yes)
 		(property "Reference" "#PWR01"
-			(at 26.67 171.45 0)
+			(at 31.75 171.45 0)
 			(effects
 				(font
@@
 		)
 		(property "Value" "GND"
-			(at 26.67 170.18 0)
+			(at 31.75 170.18 0)
 			(effects
 				(font
@@
 		)
 		(property "Footprint" ""
-			(at 26.67 165.1 0)
+			(at 31.75 165.1 0)
 			(effects
 				(font
@@
 		)
 		(property "Datasheet" ""
-			(at 26.67 165.1 0)
+			(at 31.75 165.1 0)
 			(effects
 				(font
@@
 		)
 		(property "Description" "Power symbol creates a global label with name \"GND\" , ground"
-			(at 26.67 165.1 0)
+			(at 31.75 165.1 0)
 			(effects
 				(font
@@
 	(symbol
 		(lib_id "power:PWR_FLAG")
-		(at 34.29 160.02 0)
+		(at 39.37 160.02 0)
 		(unit 1)
 		(exclude_from_sim no)
@@
 		(fields_autoplaced yes)
 		(property "Reference" "#FLG02"
-			(at 34.29 158.115 0)
+			(at 39.37 158.115 0)
 			(effects
 				(font
@@
 		)
 		(property "Value" "PWR_FLAG"
-			(at 34.29 154.94 0)
+			(at 39.37 154.94 0)
 			(effects
 				(font
@@
 		)
 		(property "Footprint" ""
-			(at 34.29 160.02 0)
+			(at 39.37 160.02 0)
 			(effects
 				(font
@@
 		)
 		(property "Datasheet" "~"
-			(at 34.29 160.02 0)
+			(at 39.37 160.02 0)
 			(effects
 				(font
@@
 		)
 		(property "Description" "Special symbol for telling ERC where power comes from"
-			(at 34.29 160.02 0)
+			(at 39.37 160.02 0)
 			(effects
 				(font
@@
 	(symbol
 		(lib_id "Custom-Symbols:solar_cell_B")
-		(at 26.67 54.61 0)
+		(at 31.75 54.61 0)
 		(unit 1)
 		(exclude_from_sim no)
@@
 		(fields_autoplaced yes)
 		(property "Reference" "S3"
-			(at 21.59 54.61 0)
+			(at 26.67 54.61 0)
 			(effects
 				(font
@@
 		)
 		(property "Value" "solar_cell_B"
-			(at 18.542 60.198 0)
+			(at 23.622 60.198 0)
 			(effects
 				(font
@@
 		)
 		(property "Footprint" "Custom-Footprints:solar_cell_B"
-			(at 16.002 48.006 0)
+			(at 21.082 48.006 0)
 			(effects
 				(font
@@
 		)
 		(property "Datasheet" ""
-			(at 26.67 54.61 0)
+			(at 31.75 54.61 0)
 			(effects
 				(font
@@
 		)
 		(property "Description" ""
-			(at 26.67 54.61 0)
+			(at 31.75 54.61 0)
 			(effects
 				(font

Commit message: Added logo and name for the panel
Parts:
- renumbered C3 to C1, C4 to C2, C1 to C3, C2 to C4
Changed lines of the file:
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@@
 		(on_board yes)
 		(dnp no)
-		(property "Reference" "C2"
+		(property "Reference" "C4"
 			(at 222.25 160.528 90)
 			(effects
@@
 			(project "UHF panel minus Y"
 				(path "/89611e38-f413-4c08-96a0-5c41e307b812"
-					(reference "C2")
+					(reference "C4")
 					(unit 1)
 				)
@@
 		(dnp no)
 		(fields_autoplaced yes)
-		(property "Reference" "C1"
+		(property "Reference" "C3"
 			(at 222.25 138.43 90)
 			(effects
@@
 			(project ""
 				(path "/89611e38-f413-4c08-96a0-5c41e307b812"
-					(reference "C1")
+					(reference "C3")
 					(unit 1)
 				)
@@
 		(dnp no)
 		(fields_autoplaced yes)
-		(property "Reference" "C3"
+		(property "Reference" "C1"
 			(at 83.82 72.6439 0)
 			(effects
@@
 			(project ""
 				(path "/89611e38-f413-4c08-96a0-5c41e307b812"
-					(reference "C3")
+					(reference "C1")
 					(unit 1)
 				)
@@
 		(dnp no)
 		(fields_autoplaced yes)
-		(property "Reference" "C4"
+		(property "Reference" "C2"
 			(at 116.84 56.1339 0)
 			(effects
@@
 			(project "UHF panel minus Y"
 				(path "/89611e38-f413-4c08-96a0-5c41e307b812"
-					(reference "C4")
-					(unit 1)
-				)
+					(reference "C2")
+					(unit 1)
+				)

Commit message: Added small camera
Parts:
- added H5: MountingHole, MountingHole:MountingHole_2.1mm, symbol Mechanical:MountingHole
Other:
- note added: "Small Camera"
Changed lines of the file:
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@@
+		)
+	)
+	(text "Small Camera"
+		(exclude_from_sim no)
+		(at 74.168 123.698 0)
+		(effects
+			(font
+				(size 2.54 2.159)
+				(thickness 0.4318)
+				(bold yes)
+			)
+			(justify left bottom)
 		)
 	)
@@
 					(unit 1)
 				)
+			)
+		)
+	)
+	(symbol
+		(lib_id "Mechanical:MountingHole")
+		(at 83.82 128.27 0)
+		(unit 1)
+		(exclude_from_sim no)
+		(in_bom no)
+		(on_board yes)
+		(dnp no)
+		(fields_autoplaced yes)
+		(property "Reference" "H5"
+			(at 86.36 126.9999 0)
+			(effects
+				(font
+					(size 1.27 1.27)
+				)
+				(justify left)
+			)
+		)
+		(property "Value" "MountingHole"
+			(at 86.36 129.5399 0)
+			(effects
+				(font
+					(size 1.27 1.27)
+				)
+				(justify left)
+			)
+		)
+		(property "Footprint" "MountingHole:MountingHole_2.1mm"
+			(at 83.82 128.27 0)
+			(effects
+				(font
+					(size 1.27 1.27)
+				)
+				(hide yes)
+			)
+		)
+		(property "Datasheet" "~"
+			(at 83.82 128.27 0)
+			(effects
+				(font
+					(size 1.27 1.27)
+				)
+				(hide yes)
+			)
+		)
+		(property "Description" "Mounting Hole without connection"
+			(at 83.82 128.27 0)
+			(effects
+				(font
+					(size 1.27 1.27)
+				)
+				(hide yes)
+			)
+		)
+		(instances
+			(project ""
+				(path "/89611e38-f413-4c08-96a0-5c41e307b812"
+					(reference "H5")
+					(unit 1)
+				)
